File: Hardware/KiCad/16_PACK_BUS_AND_DISCHARGE.kicad_sch (KiCad schematic)
At the start: 0 parts

Commit message: hardware: add PACK_BUS symbol skeleton zones
Other:
- note added: "16_PACK_BUS_AND_DISCHARGE - SYMBOL SKELETON ZONES This sheet reserves text-only zones for future PACK_BUS schematic symbols. BFE1_SW_OUT and BFE2_SW_OUT combine only at PACK_BUS_NODE on PCB-A. PACK_BUS fanout goes to CRIT, P12, P5 and LIGHT branches by star wiring or calculated bus. No K_MAIN is introduced. No high-current feed-through through PCB-B."
- note added: "PLACEHOLDER ZONE: J16_PACK_BUS_FANOUT_TBD Future connector/busbar/wire group for PACK_BUS_TO_CRIT, PACK_BUS_TO_P12, PACK_BUS_TO_P5 and PACK_BUS_TO_LIGHT. Physical connector family, current rating, wire section and pin count remain TBD."
- note added: "PLACEHOLDER ZONE: NODE16_PACK_BUS_JOIN_TBD Future schematic point for joining BFE1_SW_OUT and BFE2_SW_OUT into PACK_BUS_NODE. Must preserve independent branch diagnostics and reverse-current policy. No central mechanical K_MAIN shall be added here."
- note added: "PLACEHOLDER ZONE: SW16_PACK_BUS_DISCHARGE_TBD Future controlled discharge element for HARD_OFF verification. Sizing, energy, timeout, thermal limits and diagnostic feedback remain TBD. Discharge control must not become a hidden always-on load."
- note removed: "16_PACK_BUS_AND_DISCHARGE - LEVEL B FUNCTIONAL NETS Inputs from BFE branches: BFE1_SW_OUT and BFE2_SW_OUT. These join the common PACK_BUS_NODE only after MAIN_SW1/MAIN_SW2 functional boundaries. PACK_BUS is then exported as separate fanout groups to CRIT, 12V, 5V and LIGHT modules."
- note removed: "DISCHARGE FUNCTION PACK_BUS_DISCHARGE_EN commands the controlled discharge path. DIAG_PACK_BUS_V and DIAG_PACK_BUS_DISCH_STATUS report voltage and discharge state to PCB-B. Discharge shall be used by HARD_OFF after loads are removed and K_BAT hold loops are opened."
- note removed: "SAFE-STATE RULES No central K_MAIN is allowed. PCB-B_CTRL_RESERVE must not be a high-current feed-through for PACK_BUS. PACK_BUS discharge element sizing, energy, timeout and thermal limits remain TBD. Do not add always-on loads here without CRIT/EMG budget analysis."
Changed lines of the file:
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@@
 		(title "16_PACK_BUS_AND_DISCHARGE - PACK_BUS creation")
 		(date "2026-07-15")
-		(rev "B1")
+		(rev "C1")
 		(company "Gonoboben/plataVM")
-		(comment 1 "Architecture Level B: PACK_BUS net groups and discharge logic")
-		(comment 2 "No K_MAIN, no discharge component values, no busbar/wire gauge selected")
+		(comment 1 "Symbol skeleton: PACK_BUS join, fanout and discharge placeholders")
+		(comment 2 "Text-only placeholders; no real components, footprints or BOM part numbers")
 	)
-	(text "16_PACK_BUS_AND_DISCHARGE - LEVEL B FUNCTIONAL NETS\nInputs from BFE branches: BFE1_SW_OUT and BFE2_SW_OUT.\nThese join the common PACK_BUS_NODE only after MAIN_SW1/MAIN_SW2 functional boundaries.\nPACK_BUS is then exported as separate fanout groups to CRIT, 12V, 5V and LIGHT modules."
+	(text "16_PACK_BUS_AND_DISCHARGE - SYMBOL SKELETON ZONES\nThis sheet reserves text-only zones for future PACK_BUS schematic symbols.\nBFE1_SW_OUT and BFE2_SW_OUT combine only at PACK_BUS_NODE on PCB-A.\nPACK_BUS fanout goes to CRIT, P12, P5 and LIGHT branches by star wiring or calculated bus.\nNo K_MAIN is introduced. No high-current feed-through through PCB-B."
 		(exclude_from_sim no)
-		(at 12 18 0)
-		(effects (font (size 1.35 1.35)) (justify left))
+		(at 12 16 0)
+		(effects (font (size 1.3 1.3)) (justify left))
 		(uuid "bfe-lb-00000016-0000-4000-8000-000000000101")
 	)
-	(text "DISCHARGE FUNCTION\nPACK_BUS_DISCHARGE_EN commands the controlled discharge path.\nDIAG_PACK_BUS_V and DIAG_PACK_BUS_DISCH_STATUS report voltage and discharge state to PCB-B.\nDischarge shall be used by HARD_OFF after loads are removed and K_BAT hold loops are opened."
+	(text "PLACEHOLDER ZONE: NODE16_PACK_BUS_JOIN_TBD\nFuture schematic point for joining BFE1_SW_OUT and BFE2_SW_OUT into PACK_BUS_NODE.\nMust preserve independent branch diagnostics and reverse-current policy.\nNo central mechanical K_MAIN shall be added here."
 		(exclude_from_sim no)
-		(at 12 78 0)
-		(effects (font (size 1.3 1.3)) (justify left))
+		(at 12 70 0)
+		(effects (font (size 1.22 1.22)) (justify left))
 		(uuid "bfe-lb-00000016-0000-4000-8000-000000000102")
 	)
-	(text "SAFE-STATE RULES\nNo central K_MAIN is allowed.\nPCB-B_CTRL_RESERVE must not be a high-current feed-through for PACK_BUS.\nPACK_BUS discharge element sizing, energy, timeout and thermal limits remain TBD.\nDo not add always-on loads here without CRIT/EMG budget analysis."
+	(text "PLACEHOLDER ZONE: J16_PACK_BUS_FANOUT_TBD\nFuture connector/busbar/wire group for PACK_BUS_TO_CRIT, PACK_BUS_TO_P12, PACK_BUS_TO_P5 and PACK_BUS_TO_LIGHT.\nPhysical connector family, current rating, wire section and pin count remain TBD."
 		(exclude_from_sim no)
-		(at 12 138 0)
-		(effects (font (size 1.25 1.25)) (justify left))
+		(at 12 116 0)
+		(effects (font (size 1.22 1.22)) (justify left))
 		(uuid "bfe-lb-00000016-0000-4000-8000-000000000103")
 	)
-	(hierarchical_label "BFE1_SW_OUT" (shape passive) (exclude_from_sim no) (at 128 48 0) (effects (font (size 1.15 1.15)) (justify left)) (uuid "bfe-lb-00000016-0000-4000-8000-000000000201"))
-	(hierarchical_label "BFE2_SW_OUT" (shape passive) (exclude_from_sim no) (at 128 60 0) (effects (font (size 1.15 1.15)) (justify left)) (uuid "bfe-lb-00000016-0000-4000-8000-000000000202"))
-	(hierarchical_label "PACK_BUS_NODE" (shape passive) (exclude_from_sim no) (at 128 78 0) (effects (font (size 1.15 1.15)) (justify left)) (uuid "bfe-lb-00000016-0000-4000-8000-000000000203"))
-	(hierarchical_label "PACK_BUS_TO_CRIT" (shape passive) (exclude_from_sim no) (at 128 96 0) (effects (font (size 1.15 1.15)) (justify left)) (uuid "bfe-lb-00000016-0000-4000-8000-000000000204"))
-	(hierarchical_label "PACK_BUS_TO_P12" (shape passive) (exclude_from_sim no) (at 128 108 0) (effects (font (size 1.15 1.15)) (justify left)) (uuid "bfe-lb-00000016-0000-4000-8000-000000000205"))
-	(hierarchical_label "PACK_BUS_TO_P5" (shape passive) (exclude_from_sim no) (at 128 120 0) (effects (font (size 1.15 1.15)) (justify left)) (uuid "bfe-lb-00000016-0000-4000-8000-000000000206"))
-	(hierarchical_label "PACK_BUS_TO_LIGHT" (shape passive) (exclude_from_sim no) (at 128 132 0) (effects (font (size 1.15 1.15)) (justify left)) (uuid "bfe-lb-00000016-0000-4000-8000-000000000207"))
-	(hierarchical_label "PACK_BUS_DISCHARGE_EN" (shape input) (exclude_from_sim no) (at 128 158 0) (effects (font (size 1.15 1.15)) (justify left)) (uuid "bfe-lb-00000016-0000-4000-8000-000000000208"))
-	(hierarchical_label "DIAG_PACK_BUS_V" (shape output) (exclude_from_sim no) (at 128 170 0) (effects (font (size 1.15 1.15)) (justify left)) (uuid "bfe-lb-00000016-0000-4000-8000-000000000209"))
-	(hierarchical_label "DIAG_PACK_BUS_DISCH_STATUS" (shape output) (exclude_from_sim no) (at 128 182 0) (effects (font (size 1.15 1.15)) (justify left)) (uuid "bfe-lb-00000016-0000-4000-8000-000000000210"))
+	(text "PLACEHOLDER ZONE: SW16_PACK_BUS_DISCHARGE_TBD\nFuture controlled discharge element for HARD_OFF verification.\nSizing, energy, timeout, thermal limits and diagnostic feedback remain TBD.\nDischarge control must not become a hidden always-on load."
+		(exclude_from_sim no)
+		(at 12 160 0)
+		(effects (font (size 1.22 1.22)) (justify left))
+		(uuid "bfe-lb-00000016-0000-4000-8000-000000000104")
+	)
+	(hierarchical_label "BFE1_SW_OUT" (shape passive) (exclude_from_sim no) (at 150 62 0) (effects (font (size 1.1 1.1)) (justify left)) (uuid "bfe-lb-00000016-0000-4000-8000-000000000201"))
+	(hierarchical_label "BFE2_SW_OUT" (shape passive) (exclude_from_sim no) (at 150 70 0) (effects (font (size 1.1 1.1)) (justify left)) (uuid "bfe-lb-00000016-0000-4000-8000-000000000202"))
+	(hierarchical_label "PACK_BUS_NODE" (shape passive) (exclude_from_sim no) (at 150 82 0) (effects (font (size 1.1 1.1)) (justify left)) (uuid "bfe-lb-00000016-0000-4000-8000-000000000203"))
+	(hierarchical_label "PACK_BUS_TO_CRIT" (shape passive) (exclude_from_sim no) (at 150 126 0) (effects (font (size 1.1 1.1)) (justify left)) (uuid "bfe-lb-00000016-0000-4000-8000-000000000204"))
+	(hierarchical_label "PACK_BUS_TO_P12" (shape passive) (exclude_from_sim no) (at 150 134 0) (effects (font (size 1.1 1.1)) (justify left)) (uuid "bfe-lb-00000016-0000-4000-8000-000000000205"))
+	(hierarchical_label "PACK_BUS_TO_P5" (shape passive) (exclude_from_sim no) (at 150 142 0) (effects (font (size 1.1 1.1)) (justify left)) (uuid "bfe-lb-00000016-0000-4000-8000-000000000206"))
+	(hierarchical_label "PACK_BUS_TO_LIGHT" (shape passive) (exclude_from_sim no) (at 150 150 0) (effects (font (size 1.1 1.1)) (justify left)) (uuid "bfe-lb-00000016-0000-4000-8000-000000000207"))
+	(hierarchical_label "PACK_BUS_DISCHARGE_EN" (shape input) (exclude_from_sim no) (at 150 176 0) (effects (font (size 1.1 1.1)) (justify left)) (uuid "bfe-lb-00000016-0000-4000-8000-000000000208"))
+	(hierarchical_label "DIAG_PACK_BUS_V" (shape output) (exclude_from_sim no) (at 150 188 0) (effects (font (size 1.1 1.1)) (justify left)) (uuid "bfe-lb-00000016-0000-4000-8000-000000000209"))
+	(hierarchical_label "DIAG_PACK_BUS_DISCH_STATUS" (shape output) (exclude_from_sim no) (at 150 196 0) (effects (font (size 1.1 1.1)) (justify left)) (uuid "bfe-lb-00000016-0000-4000-8000-000000000210"))
 )
