File: Hardware/KiCad/13_MAIN_PATH_1.kicad_sch (KiCad schematic)
At the start: 0 parts

Commit message: hardware: refine MAIN_PATH_1 level B
Other:
- note added: "13_MAIN_PATH_1 - LEVEL B FUNCTIONAL NETS BAT1_TO_MAIN_PATH enters the BFE_1 electronic path. MAIN_SW1_INPUT and MAIN_SW1_OUTPUT are functional nodes around MAIN_SW1_TBD. MAIN_SW1_OUTPUT becomes BFE1_SW_OUT and later joins PACK_BUS_NODE on sheet 16."
- note added: "CONTROL AND SAFE STATE CTRL_MAIN_SW1_EN enables the branch only when allowed by firmware and hardware safety. MAIN_SW1_SAFE_OFF and EXT_KILL_HW_CHAIN must force the branch OFF independent of normal load commands. Reverse current policy, precharge/inrush handling and SOA remain TBD."
- note added: "DIAGNOSTICS DIAG_MAIN1_I, DIAG_MAIN1_VIN, DIAG_MAIN1_VOUT and DIAG_MAIN1_FAULT are grouped outputs to PCB-B. Measurement topology and ADC frontend remain TBD. Do not add K_MAIN or route all PACK_BUS current through PCB-B_CTRL_RESERVE."
- note removed: "13_MAIN_PATH_1 - FUNCTIONAL PATH BAT1_TO_MAIN_PATH -> input protection / current measurement TBD -> MAIN_SW1 -> PACK_BUS contribution. MAIN_SW1 is an electronic power path controlled by PCB-B and disabled by EXT_KILL/HARD_OFF. This sheet does not select MOSFETs, eFuse, ideal-diode controller, current sensor or thermal solution."
- note removed: "OPEN ITEMS MAIN_SW1 topology, reverse-current policy, SOA, current-sense method, thermal limits and fault timing remain TBD. Do not add K_MAIN. Do not route all PACK_BUS current through PCB-B_CTRL_RESERVE."
- note removed: "REQUIRED BEHAVIOR - allow controlled connection of BAT1 branch to PACK_BUS; - support load-shedding before mechanical K_BAT1 opens; - report voltage/current/fault state to PCB-B; - fail toward OFF under EXT_KILL and critical faults; - preserve independent branch behavior against BFE_2."
Changed lines of the file:
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@@
 	(generator "eeschema")
 	(generator_version "10.0")
-	(uuid "bfe-dh-00000013-0000-4000-8000-000000000013")
+	(uuid "bfe-lb-00000013-0000-4000-8000-000000000013")
 	(paper "A3")
 	(title_block
 		(title "13_MAIN_PATH_1 - BFE_1 main electronic path")
 		(date "2026-07-15")
-		(rev "A1")
+		(rev "B1")
 		(company "Gonoboben/plataVM")
-		(comment 1 "Architecture Level A: MAIN_SW1 functional boundary")
-		(comment 2 "No MAIN_SW1 topology or component selected")
+		(comment 1 "Architecture Level B: MAIN_SW1 control, diagnostics and safe-state nets")
+		(comment 2 "No MAIN_SW1 topology, MOSFET, eFuse or current sensor selected")
 	)
-	(text "13_MAIN_PATH_1 - FUNCTIONAL PATH\nBAT1_TO_MAIN_PATH -> input protection / current measurement TBD -> MAIN_SW1 -> PACK_BUS contribution.\nMAIN_SW1 is an electronic power path controlled by PCB-B and disabled by EXT_KILL/HARD_OFF.\nThis sheet does not select MOSFETs, eFuse, ideal-diode controller, current sensor or thermal solution."
+	(text "13_MAIN_PATH_1 - LEVEL B FUNCTIONAL NETS\nBAT1_TO_MAIN_PATH enters the BFE_1 electronic path.\nMAIN_SW1_INPUT and MAIN_SW1_OUTPUT are functional nodes around MAIN_SW1_TBD.\nMAIN_SW1_OUTPUT becomes BFE1_SW_OUT and later joins PACK_BUS_NODE on sheet 16."
 		(exclude_from_sim no)
 		(at 12 18 0)
-		(effects (font (size 1.45 1.45)) (justify left))
-		(uuid "bfe-dh-00000013-0000-4000-8000-000000000101")
+		(effects (font (size 1.35 1.35)) (justify left))
+		(uuid "bfe-lb-00000013-0000-4000-8000-000000000101")
 	)
-	(text "REQUIRED BEHAVIOR\n- allow controlled connection of BAT1 branch to PACK_BUS;\n- support load-shedding before mechanical K_BAT1 opens;\n- report voltage/current/fault state to PCB-B;\n- fail toward OFF under EXT_KILL and critical faults;\n- preserve independent branch behavior against BFE_2."
+	(text "CONTROL AND SAFE STATE\nCTRL_MAIN_SW1_EN enables the branch only when allowed by firmware and hardware safety.\nMAIN_SW1_SAFE_OFF and EXT_KILL_HW_CHAIN must force the branch OFF independent of normal load commands.\nReverse current policy, precharge/inrush handling and SOA remain TBD."
 		(exclude_from_sim no)
 		(at 12 78 0)
-		(effects (font (size 1.35 1.35)) (justify left))
-		(uuid "bfe-dh-00000013-0000-4000-8000-000000000102")
+		(effects (font (size 1.3 1.3)) (justify left))
+		(uuid "bfe-lb-00000013-0000-4000-8000-000000000102")
 	)
-	(text "OPEN ITEMS\nMAIN_SW1 topology, reverse-current policy, SOA, current-sense method, thermal limits and fault timing remain TBD.\nDo not add K_MAIN. Do not route all PACK_BUS current through PCB-B_CTRL_RESERVE."
+	(text "DIAGNOSTICS\nDIAG_MAIN1_I, DIAG_MAIN1_VIN, DIAG_MAIN1_VOUT and DIAG_MAIN1_FAULT are grouped outputs to PCB-B.\nMeasurement topology and ADC frontend remain TBD.\nDo not add K_MAIN or route all PACK_BUS current through PCB-B_CTRL_RESERVE."
 		(exclude_from_sim no)
 		(at 12 140 0)
-		(effects (font (size 1.3 1.3)) (justify left))
-		(uuid "bfe-dh-00000013-0000-4000-8000-000000000103")
+		(effects (font (size 1.25 1.25)) (justify left))
+		(uuid "bfe-lb-00000013-0000-4000-8000-000000000103")
 	)
-	(hierarchical_label "BAT1_TO_MAIN_PATH" (shape passive) (exclude_from_sim no) (at 120 52 0) (effects (font (size 1.15 1.15)) (justify left)) (uuid "bfe-dh-00000013-0000-4000-8000-000000000201"))
-	(hierarchical_label "MAIN_SW1_TO_PACK_BUS" (shape passive) (exclude_from_sim no) (at 120 64 0) (effects (font (size 1.15 1.15)) (justify left)) (uuid "bfe-dh-00000013-0000-4000-8000-000000000202"))
-	(hierarchical_label "CTRL_MAIN_SW1_EN" (shape input) (exclude_from_sim no) (at 120 96 0) (effects (font (size 1.15 1.15)) (justify left)) (uuid "bfe-dh-00000013-0000-4000-8000-000000000203"))
-	(hierarchical_label "DIAG_MAIN_PATH_1" (shape output) (exclude_from_sim no) (at 120 108 0) (effects (font (size 1.15 1.15)) (justify left)) (uuid "bfe-dh-00000013-0000-4000-8000-000000000204"))
+	(hierarchical_label "BAT1_TO_MAIN_PATH" (shape passive) (exclude_from_sim no) (at 126 48 0) (effects (font (size 1.15 1.15)) (justify left)) (uuid "bfe-lb-00000013-0000-4000-8000-000000000201"))
+	(hierarchical_label "MAIN_SW1_INPUT" (shape passive) (exclude_from_sim no) (at 126 60 0) (effects (font (size 1.15 1.15)) (justify left)) (uuid "bfe-lb-00000013-0000-4000-8000-000000000202"))
+	(hierarchical_label "MAIN_SW1_OUTPUT" (shape passive) (exclude_from_sim no) (at 126 72 0) (effects (font (size 1.15 1.15)) (justify left)) (uuid "bfe-lb-00000013-0000-4000-8000-000000000203"))
+	(hierarchical_label "BFE1_SW_OUT" (shape passive) (exclude_from_sim no) (at 126 84 0) (effects (font (size 1.15 1.15)) (justify left)) (uuid "bfe-lb-00000013-0000-4000-8000-000000000204"))
+	(hierarchical_label "CTRL_MAIN_SW1_EN" (shape input) (exclude_from_sim no) (at 126 108 0) (effects (font (size 1.15 1.15)) (justify left)) (uuid "bfe-lb-00000013-0000-4000-8000-000000000205"))
+	(hierarchical_label "MAIN_SW1_SAFE_OFF" (shape input) (exclude_from_sim no) (at 126 120 0) (effects (font (size 1.15 1.15)) (justify left)) (uuid "bfe-lb-00000013-0000-4000-8000-000000000206"))
+	(hierarchical_label "EXT_KILL_HW_CHAIN" (shape input) (exclude_from_sim no) (at 126 132 0) (effects (font (size 1.15 1.15)) (justify left)) (uuid "bfe-lb-00000013-0000-4000-8000-000000000207"))
+	(hierarchical_label "DIAG_MAIN1_I" (shape output) (exclude_from_sim no) (at 126 158 0) (effects (font (size 1.15 1.15)) (justify left)) (uuid "bfe-lb-00000013-0000-4000-8000-000000000208"))
+	(hierarchical_label "DIAG_MAIN1_VIN" (shape output) (exclude_from_sim no) (at 126 170 0) (effects (font (size 1.15 1.15)) (justify left)) (uuid "bfe-lb-00000013-0000-4000-8000-000000000209"))
+	(hierarchical_label "DIAG_MAIN1_VOUT" (shape output) (exclude_from_sim no) (at 126 182 0) (effects (font (size 1.15 1.15)) (justify left)) (uuid "bfe-lb-00000013-0000-4000-8000-000000000210"))
+	(hierarchical_label "DIAG_MAIN1_FAULT" (shape output) (exclude_from_sim no) (at 126 194 0) (effects (font (size 1.15 1.15)) (justify left)) (uuid "bfe-lb-00000013-0000-4000-8000-000000000211"))
 )
