File: Hardware/KiCad/15_DECK_BALANCE.kicad_sch (KiCad schematic)
At the start: 0 parts

Commit message: hardware: refine DECK_BALANCE level B
Other:
- note added: "15_DECK_BALANCE - LEVEL B FUNCTIONAL NETS Deck-side balancing is a controlled maintenance/state-machine function after work, not an always-on passive equalizer. It uses BAT1/BAT2 balance tap groups and a current-limited BALANCE_PATH_TBD. It must not bypass BMS protection or replace branch fault handling."
- note added: "CONTROL AND ABORT BALANCE_ARM permits the function only in allowed system states. BALANCE_SW1_EN and BALANCE_SW2_EN command branch-side switching boundaries. BALANCE_ABORT and EXT_KILL_HW_CHAIN must disable the path. Balance current, delta-V limits, duration and thermal model remain TBD."
- note added: "DIAGNOSTICS DIAG_BALANCE_I, DIAG_BALANCE_TEMP and DIAG_BALANCE_STATUS are logical groups to PCB-B. The final circuit must provide timeout/fault logging and fail toward OFF. R_BAL, switch SOA, thermal sensor placement and protection remain TBD."
- note removed: "15_DECK_BALANCE - FUNCTIONAL PURPOSE Deck-side balancing is performed only after work / under controlled conditions. It is not an always-on passive equalizer and does not bypass BMS protection. The balance path is commanded by MCU logic and must be blocked by unsafe states."
- note removed: "FUNCTIONAL BLOCKS - BALANCE_SW1 / BALANCE_SW2 command boundary; - R_BAL / current-limited equalization path TBD; - voltage/current monitoring dependency; - firmware interlock dependency; - thermal timeout and fault logging dependency."
- note removed: "OPEN ITEMS Balance current, allowed delta-V, resistor power, switch SOA, thermal sensor placement, duration and abort logic remain TBD. Do not use balancing as a substitute for BMS protection or main branch fault handling."
Changed lines of the file:
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@@
 	(generator "eeschema")
 	(generator_version "10.0")
-	(uuid "bfe-dh-00000015-0000-4000-8000-000000000015")
+	(uuid "bfe-lb-00000015-0000-4000-8000-000000000015")
 	(paper "A3")
 	(title_block
 		(title "15_DECK_BALANCE - controlled equalization path")
 		(date "2026-07-15")
-		(rev "A1")
+		(rev "B1")
 		(company "Gonoboben/plataVM")
-		(comment 1 "Architecture Level A: deck-side balance functional boundary")
-		(comment 2 "No resistor, switch or control topology selected")
+		(comment 1 "Architecture Level B: balance control, measurement dependency and abort nets")
+		(comment 2 "No resistor, switch, current value or thermal solution selected")
 	)
-	(text "15_DECK_BALANCE - FUNCTIONAL PURPOSE\nDeck-side balancing is performed only after work / under controlled conditions.\nIt is not an always-on passive equalizer and does not bypass BMS protection.\nThe balance path is commanded by MCU logic and must be blocked by unsafe states."
+	(text "15_DECK_BALANCE - LEVEL B FUNCTIONAL NETS\nDeck-side balancing is a controlled maintenance/state-machine function after work, not an always-on passive equalizer.\nIt uses BAT1/BAT2 balance tap groups and a current-limited BALANCE_PATH_TBD.\nIt must not bypass BMS protection or replace branch fault handling."
 		(exclude_from_sim no)
 		(at 12 18 0)
-		(effects (font (size 1.45 1.45)) (justify left))
-		(uuid "bfe-dh-00000015-0000-4000-8000-000000000101")
+		(effects (font (size 1.35 1.35)) (justify left))
+		(uuid "bfe-lb-00000015-0000-4000-8000-000000000101")
 	)
-	(text "FUNCTIONAL BLOCKS\n- BALANCE_SW1 / BALANCE_SW2 command boundary;\n- R_BAL / current-limited equalization path TBD;\n- voltage/current monitoring dependency;\n- firmware interlock dependency;\n- thermal timeout and fault logging dependency."
+	(text "CONTROL AND ABORT\nBALANCE_ARM permits the function only in allowed system states.\nBALANCE_SW1_EN and BALANCE_SW2_EN command branch-side switching boundaries.\nBALANCE_ABORT and EXT_KILL_HW_CHAIN must disable the path.\nBalance current, delta-V limits, duration and thermal model remain TBD."
 		(exclude_from_sim no)
-		(at 12 78 0)
-		(effects (font (size 1.35 1.35)) (justify left))
-		(uuid "bfe-dh-00000015-0000-4000-8000-000000000102")
+		(at 12 82 0)
+		(effects (font (size 1.25 1.25)) (justify left))
+		(uuid "bfe-lb-00000015-0000-4000-8000-000000000102")
 	)
-	(text "OPEN ITEMS\nBalance current, allowed delta-V, resistor power, switch SOA, thermal sensor placement, duration and abort logic remain TBD.\nDo not use balancing as a substitute for BMS protection or main branch fault handling."
+	(text "DIAGNOSTICS\nDIAG_BALANCE_I, DIAG_BALANCE_TEMP and DIAG_BALANCE_STATUS are logical groups to PCB-B.\nThe final circuit must provide timeout/fault logging and fail toward OFF.\nR_BAL, switch SOA, thermal sensor placement and protection remain TBD."
 		(exclude_from_sim no)
-		(at 12 140 0)
-		(effects (font (size 1.3 1.3)) (justify left))
-		(uuid "bfe-dh-00000015-0000-4000-8000-000000000103")
+		(at 12 152 0)
+		(effects (font (size 1.25 1.25)) (justify left))
+		(uuid "bfe-lb-00000015-0000-4000-8000-000000000103")
 	)
-	(hierarchical_label "BALANCE_PATH_BAT1" (shape passive) (exclude_from_sim no) (at 120 56 0) (effects (font (size 1.15 1.15)) (justify left)) (uuid "bfe-dh-00000015-0000-4000-8000-000000000201"))
-	(hierarchical_label "BALANCE_PATH_BAT2" (shape passive) (exclude_from_sim no) (at 120 68 0) (effects (font (size 1.15 1.15)) (justify left)) (uuid "bfe-dh-00000015-0000-4000-8000-000000000202"))
-	(hierarchical_label "CTRL_BALANCE_SW1_EN" (shape input) (exclude_from_sim no) (at 120 102 0) (effects (font (size 1.15 1.15)) (justify left)) (uuid "bfe-dh-00000015-0000-4000-8000-000000000203"))
-	(hierarchical_label "CTRL_BALANCE_SW2_EN" (shape input) (exclude_from_sim no) (at 120 114 0) (effects (font (size 1.15 1.15)) (justify left)) (uuid "bfe-dh-00000015-0000-4000-8000-000000000204"))
-	(hierarchical_label "DIAG_BALANCE" (shape output) (exclude_from_sim no) (at 120 126 0) (effects (font (size 1.15 1.15)) (justify left)) (uuid "bfe-dh-00000015-0000-4000-8000-000000000205"))
+	(hierarchical_label "BALANCE_TAP_BAT1" (shape passive) (exclude_from_sim no) (at 128 50 0) (effects (font (size 1.15 1.15)) (justify left)) (uuid "bfe-lb-00000015-0000-4000-8000-000000000201"))
+	(hierarchical_label "BALANCE_TAP_BAT2" (shape passive) (exclude_from_sim no) (at 128 62 0) (effects (font (size 1.15 1.15)) (justify left)) (uuid "bfe-lb-00000015-0000-4000-8000-000000000202"))
+	(hierarchical_label "BALANCE_PATH_TBD" (shape passive) (exclude_from_sim no) (at 128 74 0) (effects (font (size 1.15 1.15)) (justify left)) (uuid "bfe-lb-00000015-0000-4000-8000-000000000203"))
+	(hierarchical_label "BALANCE_ARM" (shape input) (exclude_from_sim no) (at 128 98 0) (effects (font (size 1.15 1.15)) (justify left)) (uuid "bfe-lb-00000015-0000-4000-8000-000000000204"))
+	(hierarchical_label "BALANCE_SW1_EN" (shape input) (exclude_from_sim no) (at 128 110 0) (effects (font (size 1.15 1.15)) (justify left)) (uuid "bfe-lb-00000015-0000-4000-8000-000000000205"))
+	(hierarchical_label "BALANCE_SW2_EN" (shape input) (exclude_from_sim no) (at 128 122 0) (effects (font (size 1.15 1.15)) (justify left)) (uuid "bfe-lb-00000015-0000-4000-8000-000000000206"))
+	(hierarchical_label "BALANCE_ABORT" (shape input) (exclude_from_sim no) (at 128 134 0) (effects (font (size 1.15 1.15)) (justify left)) (uuid "bfe-lb-00000015-0000-4000-8000-000000000207"))
+	(hierarchical_label "EXT_KILL_HW_CHAIN" (shape input) (exclude_from_sim no) (at 128 146 0) (effects (font (size 1.15 1.15)) (justify left)) (uuid "bfe-lb-00000015-0000-4000-8000-000000000208"))
+	(hierarchical_label "DIAG_BALANCE_I" (shape output) (exclude_from_sim no) (at 128 172 0) (effects (font (size 1.15 1.15)) (justify left)) (uuid "bfe-lb-00000015-0000-4000-8000-000000000209"))
+	(hierarchical_label "DIAG_BALANCE_TEMP" (shape output) (exclude_from_sim no) (at 128 184 0) (effects (font (size 1.15 1.15)) (justify left)) (uuid "bfe-lb-00000015-0000-4000-8000-000000000210"))
+	(hierarchical_label "DIAG_BALANCE_STATUS" (shape output) (exclude_from_sim no) (at 128 196 0) (effects (font (size 1.15 1.15)) (justify left)) (uuid "bfe-lb-00000015-0000-4000-8000-000000000211"))
 )
