File: Hardware/KiCad/23_MCU_CORE.kicad_sch (KiCad schematic)
At the start: 0 parts

Commit message: hardware: align PCB-B CTRL_RESERVE interfaces
Merge PCB-B interface consistency fixes after verifying canonical names, diagnostics, and independent EXT_KILL final actions.
Other:
- note added: "NORMAL CONTROL / DIAGNOSTICS MCU_TO_CONTROL_IO and CONTROL_IO_TO_MCU are logical boundaries only; they do not select parallel, muxed, SPI, I2C or other internal transport. EMG, watchdog, fault-latch and RS-485 link states are observation inputs for logging. All externally visible commands require defined defaults during reset, brownout and unpowered conditions."
- note added: "SAFETY LIMIT EXT_KILL_EVENT_STATUS may be logged by firmware, but firmware cannot block, postpone or clear EXT_KILL_LATCHED. CONTROLLED_SHUTDOWN_REQ requests an orderly critical-domain shutdown; it does not replace hardware OFF. BMS recovery or critical-rail recovery must not cause automatic energization of K_BATx."
- note removed: "NORMAL CONTROL / DIAGNOSTICS MCU_TO_CONTROL_IO and CONTROL_IO_TO_MCU are logical boundaries only; they do not select parallel, muxed, SPI, I2C or other internal transport. The MCU may issue normal OFF commands and safe-state requests. All externally visible commands require defined defaults during reset, brownout and unpowered conditions."
- note removed: "SAFETY LIMIT EXT_KILL_EVENT_STATUS may be logged by firmware, but firmware cannot block, postpone or clear EXT_KILL_LATCHED. Watchdog/supervisor may reset or contain the MCU independently. BMS recovery or critical-rail recovery must not cause automatic energization of K_BATx."
Changed lines of the file:
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@@
 		(title "23_MCU_CORE - control processor functional boundary")
 		(date "2026-07-15")
-		(rev "B0")
+		(rev "B1")
 		(company "Gonoboben/plataVM")
-		(comment 1 "Architecture Level A/B: MCU core, logging and logical interface ownership")
+		(comment 1 "Interface consistency: MCU logging/status boundaries completed")
 		(comment 2 "No MCU family, clock, memory, ADC, isolation, programming connector or footprint selected")
 	)
@@
 		(uuid "ctrl-reserve-00000023-0000-4000-8000-000000000102")
 	)
-	(text "NORMAL CONTROL / DIAGNOSTICS\nMCU_TO_CONTROL_IO and CONTROL_IO_TO_MCU are logical boundaries only; they do not select parallel, muxed, SPI, I2C or other internal transport.\nThe MCU may issue normal OFF commands and safe-state requests.\nAll externally visible commands require defined defaults during reset, brownout and unpowered conditions."
+	(text "NORMAL CONTROL / DIAGNOSTICS\nMCU_TO_CONTROL_IO and CONTROL_IO_TO_MCU are logical boundaries only; they do not select parallel, muxed, SPI, I2C or other internal transport.\nEMG, watchdog, fault-latch and RS-485 link states are observation inputs for logging.\nAll externally visible commands require defined defaults during reset, brownout and unpowered conditions."
 		(exclude_from_sim no)
 		(at 12 130 0)
-		(effects (font (size 1.16 1.16)) (justify left))
+		(effects (font (size 1.14 1.14)) (justify left))
 		(uuid "ctrl-reserve-00000023-0000-4000-8000-000000000103")
 	)
-	(text "SAFETY LIMIT\nEXT_KILL_EVENT_STATUS may be logged by firmware, but firmware cannot block, postpone or clear EXT_KILL_LATCHED.\nWatchdog/supervisor may reset or contain the MCU independently.\nBMS recovery or critical-rail recovery must not cause automatic energization of K_BATx."
+	(text "SAFETY LIMIT\nEXT_KILL_EVENT_STATUS may be logged by firmware, but firmware cannot block, postpone or clear EXT_KILL_LATCHED.\nCONTROLLED_SHUTDOWN_REQ requests an orderly critical-domain shutdown; it does not replace hardware OFF.\nBMS recovery or critical-rail recovery must not cause automatic energization of K_BATx."
 		(exclude_from_sim no)
 		(at 12 198 0)
-		(effects (font (size 1.16 1.16)) (justify left))
+		(effects (font (size 1.14 1.14)) (justify left))
 		(uuid "ctrl-reserve-00000023-0000-4000-8000-000000000104")
 	)
@@
 	(hierarchical_label "RS485_LOGIC" (shape passive) (exclude_from_sim no) (at 150 190 0) (effects (font (size 1.1 1.1)) (justify left)) (uuid "ctrl-reserve-00000023-0000-4000-8000-000000000209"))
 	(hierarchical_label "SERVICE_DEBUG_LOGIC" (shape passive) (exclude_from_sim no) (at 150 198 0) (effects (font (size 1.1 1.1)) (justify left)) (uuid "ctrl-reserve-00000023-0000-4000-8000-000000000210"))
-	(hierarchical_label "EXT_KILL_EVENT_STATUS" (shape input) (exclude_from_sim no) (at 150 230 0) (effects (font (size 1.1 1.1)) (justify left)) (uuid "ctrl-reserve-00000023-0000-4000-8000-000000000211"))
-	(hierarchical_label "CONTROLLED_SHUTDOWN_REQ" (shape input) (exclude_from_sim no) (at 150 238 0) (effects (font (size 1.1 1.1)) (justify left)) (uuid "ctrl-reserve-00000023-0000-4000-8000-000000000212"))
+	(hierarchical_label "EXT_KILL_EVENT_STATUS" (shape input) (exclude_from_sim no) (at 150 222 0) (effects (font (size 1.1 1.1)) (justify left)) (uuid "ctrl-reserve-00000023-0000-4000-8000-000000000211"))
+	(hierarchical_label "CONTROLLED_SHUTDOWN_REQ" (shape input) (exclude_from_sim no) (at 150 230 0) (effects (font (size 1.1 1.1)) (justify left)) (uuid "ctrl-reserve-00000023-0000-4000-8000-000000000212"))
+	(hierarchical_label "EMG_CHARGE_STATUS" (shape input) (exclude_from_sim no) (at 300 112 0) (effects (font (size 1.1 1.1)) (justify left)) (uuid "ctrl-reserve-00000023-0000-4000-8000-000000000213"))
+	(hierarchical_label "FAULT_LATCHED_STATUS" (shape input) (exclude_from_sim no) (at 300 120 0) (effects (font (size 1.1 1.1)) (justify left)) (uuid "ctrl-reserve-00000023-0000-4000-8000-000000000214"))
+	(hierarchical_label "WATCHDOG_FAULT_N" (shape input) (exclude_from_sim no) (at 300 128 0) (effects (font (size 1.1 1.1)) (justify left)) (uuid "ctrl-reserve-00000023-0000-4000-8000-000000000215"))
+	(hierarchical_label "RS485_LINK_STATUS" (shape input) (exclude_from_sim no) (at 300 136 0) (effects (font (size 1.1 1.1)) (justify left)) (uuid "ctrl-reserve-00000023-0000-4000-8000-000000000216"))
 )

Commit message: hardware: add internal CAN-FD ownership to MCU boundary
Other:
- note added: "23_MCU_CORE - PURPOSE Defines the central normal-control processor boundary on PCB-B. The MCU performs command processing, diagnostics, logging, RS-485 protocol and internal CAN-FD management. It is not required for EXT_KILL actuation or local channel protection."
- note added: "COMMUNICATION OWNERSHIP RS485_LOGIC serves the external 115200 bit/s addressed binary link. CAN_INT_LOGIC serves normal PCB-C/D/E commands, setpoints and detailed telemetry. Direct SAFE/HARD_OFF lines and board-fault summaries bypass CAN-FD data transport."
- note added: "MCU BASELINE Preliminary family: STM32G4. Final part/package follows pin count, ADC accuracy, memory and peripheral review. Required functions include independent watchdog interaction, CRC, DMA, external isolated RS-485 and one internal CAN-FD controller. No part number or footprint is selected."
- note added: "SAFETY LIMIT Firmware may log EXT_KILL and faults but cannot block or clear the hardware safety path. Communication loss must not disable local protection. BMS or critical-rail recovery cannot automatically energize K_BATx. WELDED_CONTACT and HARD_OFF_FAILED block restart."
- note removed: "23_MCU_CORE - PURPOSE Defines the normal-control processor boundary on PCB-B_CTRL_RESERVE. The MCU performs command processing, diagnostics, logging and controlled shutdown. It is not a required element in the final EXT_KILL actuation path."
- note removed: "MCU CORE FUNCTIONAL ZONE Future symbols will include the selected processor, clocking, reset, decoupling, boot configuration and required memory. Pin allocation, voltage domains, ADC strategy and communication peripherals remain TBD. No part number or package is selected at this stage."
- note removed: "NORMAL CONTROL / DIAGNOSTICS MCU_TO_CONTROL_IO and CONTROL_IO_TO_MCU are logical boundaries only; they do not select parallel, muxed, SPI, I2C or other internal transport. EMG, watchdog, fault-latch and RS-485 link states are observation inputs for logging. All externally visible commands require defined defaults during reset, brownout and unpowered conditions."
- note removed: "SAFETY LIMIT EXT_KILL_EVENT_STATUS may be logged by firmware, but firmware cannot block, postpone or clear EXT_KILL_LATCHED. CONTROLLED_SHUTDOWN_REQ requests an orderly critical-domain shutdown; it does not replace hardware OFF. BMS recovery or critical-rail recovery must not cause automatic energization of K_BATx."
