File: Hardware/KiCad/41_5V_DC_DC.kicad_sch (KiCad schematic)
At the start: 46 parts

Commit message: hardware: fix PCB-D KiCad symbol coordinate transform V1.9
Connections:
- net 5V_SYS_BUS: now also U_DCDC.26 (VOUT1), U_DCDC.5 (VOUT2), U_DCDC.6 (VCCX), U_ISENSE1.2 (SHUNT_LO), U_ISENSE2.2 (SHUNT_LO); no longer U_DCDC.15 (VCC), U_DCDC.16 (VCC), U_DCDC.35 (AGND), U_ISENSE1.1 (SHUNT_HI), U_ISENSE2.1 (SHUNT_HI)
- net 5V_SYS_EN: now also U_EN_GATE.1 (5V_SYS_EN); no longer U_EN_GATE.6 (GND)
- net AGND: now also U_DCDC.28 (FB1), U_DCDC.3 (FB2), U_DCDC.35 (AGND), U_DCDC.EP (EXPOSED_PAD), U_EN_GATE.6 (GND), U_FAULT.4 (GND), U_UVLO.2 (GND); no longer U_DCDC.18 (LO1), U_DCDC.26 (VOUT1), U_DCDC.33 (DEMB), U_EN_GATE.1 (5V_SYS_EN), U_FAULT.1 (PGOOD_OD), U_UVLO.1 (VIN_SENSE)
- net COMP_COMMON: now also U_DCDC.2 (COMP2), U_DCDC.29 (COMP1); no longer U_DCDC.19 (LOL1), U_DCDC.32 (RES)
- net CS1_FILTERED: now also U_DCDC.27 (CS1); no longer U_DCDC.34 (MODE)
- net CS2_FILTERED: now also U_DCDC.4 (CS2); no longer U_DCDC.17 (PGND1)
- net EN_RUN: now also U_DCDC.31 (EN1), U_DCDC.40 (EN2), U_FAULT.3 (EN_RUN); no longer U_DCDC.21 (SW1), U_DCDC.30 (SS1), U_FAULT.2 (UVLO_OK)
- net GH1_OFF: now also U_DCDC.23 (HOL1); no longer U_DCDC.38 (DITH)
- net GH1_ON: now also U_DCDC.22 (HO1); no longer U_DCDC.39 (SYNCOUT)
- net GH2_OFF: now also U_DCDC.8 (HOL2); no longer U_DCDC.13 (LO2)
- net GH2_ON: now also U_DCDC.9 (HO2); no longer U_DCDC.12 (LOL2)
- net GL1_OFF: now also U_DCDC.19 (LOL1); no longer U_DCDC.2 (COMP2)
- net GL1_ON: now also U_DCDC.18 (LO1); no longer U_DCDC.3 (FB2)
- net GL2_OFF: now also U_DCDC.12 (LOL2); no longer U_DCDC.9 (HO2)
- net GL2_ON: now also U_DCDC.13 (LO2); no longer U_DCDC.8 (HOL2)
- net HB1_BOOT: now also U_DCDC.20 (HB1); no longer U_DCDC.1 (SS2)
- net HB2_BOOT: now also U_DCDC.11 (HB2); no longer U_DCDC.10 (SW2)
- net NC_PG2_TESTPAD: now also TP_PG2.1, U_DCDC.7 (PG2); no longer U_DCDC.14 (PGND2)
- net P5_GROUP_HARD_OFF: now also U_EN_GATE.4 (HARD_OFF); no longer U_EN_GATE.3 (SAFE_OFF)
- net P5_GROUP_SAFE_OFF: now also U_EN_GATE.3 (SAFE_OFF); no longer U_EN_GATE.4 (HARD_OFF)
- net P5_PGOOD_OD: now also U_DCDC.24 (PG1), U_FAULT.1 (PGOOD_OD); no longer U_DCDC.37 (RT), U_FAULT.4 (GND)
- net P5_PHASE1_ISENSE: now also U_ISUM.1 (PHASE1); no longer U_ISUM.2 (PHASE2)
- net P5_PHASE2_ISENSE: now also U_ISUM.2 (PHASE2); no longer U_ISUM.1 (PHASE1)
- net PACK_BUS_P5_IN: now also Q_HS1.2 (D), Q_HS2.2 (D), U_DCDC.25 (VIN), U_EN_GATE.5 (PACK_BIAS), U_UVLO.1 (VIN_SENSE); no longer Q_HS1.3 (S), Q_HS2.3 (S), U_DCDC.36 (VDDA), U_EN_GATE.2 (UVLO_OK), U_UVLO.2 (GND)
- net PHASE1_L_OUT: now also U_ISENSE1.1 (SHUNT_HI); no longer U_ISENSE1.2 (SHUNT_LO)
- net PHASE1_SW: now also Q_HS1.3 (S), Q_LS1.2 (D), U_DCDC.21 (SW1); no longer Q_HS1.2 (D), Q_LS1.3 (S), U_DCDC.40 (EN2)
- net PHASE2_L_OUT: now also U_ISENSE2.1 (SHUNT_HI); no longer U_ISENSE2.2 (SHUNT_LO)
- net PHASE2_SW: now also Q_HS2.3 (S), Q_LS2.2 (D), U_DCDC.10 (SW2); no longer Q_HS2.2 (D), Q_LS2.3 (S), U_DCDC.11 (HB2)
- net POWER_GND: now also Q_LS1.3 (S), Q_LS2.3 (S), U_DCDC.14 (PGND2), U_DCDC.17 (PGND1); no longer Q_LS1.2 (D), Q_LS2.2 (D), U_DCDC.4 (CS2), U_DCDC.7 (PG2)
- net RES_TIMER: now also U_DCDC.32 (RES); no longer U_DCDC.29 (COMP1)
- net RT_SET: now also U_DCDC.37 (RT); no longer U_DCDC.24 (PG1)
- net SS_COMMON: now also U_DCDC.1 (SS2), U_DCDC.30 (SS1); no longer U_DCDC.20 (HB1), U_DCDC.31 (EN1)
- net SYNCOUT_TESTPAD: now also TP_SYNC.1, U_DCDC.39 (SYNCOUT); no longer U_DCDC.22 (HO1)
- net UVLO_OK: now also U_EN_GATE.2 (UVLO_OK), U_FAULT.2 (UVLO_OK); no longer U_EN_GATE.5 (PACK_BIAS), U_FAULT.3 (EN_RUN)
- net VCC_BIAS: now also U_DCDC.15 (VCC), U_DCDC.16 (VCC); no longer U_DCDC.5 (VOUT2), U_DCDC.6 (VCCX)
- net VDDA_BIAS: now also U_DCDC.33 (DEMB), U_DCDC.34 (MODE), U_DCDC.36 (VDDA), U_DCDC.38 (DITH); no longer U_DCDC.23 (HOL1), U_DCDC.25 (VIN), U_DCDC.27 (CS1), U_DCDC.28 (FB1)

Commit message: hardware: exact PCB-D discrete physical pin map V1.9
Parts:
- Q_HS1, Q_HS2, Q_LS1, Q_LS2: symbol plataVM:NMOS_POWER -> plataVM:BUK9Y6R0_60E_LFPAK56
- RSH1, RSH2: symbol plataVM:R -> plataVM:WSK2512_4T_KELVIN
Connections:
- net 5V_SYS_BUS: now also RSH1.I2, RSH2.I2; no longer C_CS1.2, C_CS2.2, RSH1.2, RSH2.2, U_DCDC.26 (VOUT1), U_DCDC.5 (VOUT2), U_ISENSE1.2 (SHUNT_LO), U_ISENSE2.2 (SHUNT_LO)
- net PACK_BUS_P5_IN: now also Q_HS1.mb (D), Q_HS2.mb (D); no longer Q_HS1.2 (D), Q_HS2.2 (D)
- net PHASE1_L_OUT: now also RSH1.I1; no longer RSH1.1, R_CS1.1, U_ISENSE1.1 (SHUNT_HI)
- net PHASE1_SW: now also Q_HS1.1 (S), Q_HS1.2 (S), Q_LS1.mb (D); no longer Q_LS1.2 (D)
- net PHASE2_L_OUT: now also RSH2.I1; no longer RSH2.1, R_CS2.1, U_ISENSE2.1 (SHUNT_HI)
- net PHASE2_SW: now also Q_HS2.1 (S), Q_HS2.2 (S), Q_LS2.mb (D); no longer Q_LS2.2 (D)
- net POWER_GND: now also Q_LS1.1 (S), Q_LS1.2 (S), Q_LS2.1 (S), Q_LS2.2 (S)
- net Q_HS1_GATE: now also Q_HS1.4 (G); no longer Q_HS1.1 (G)
- net Q_HS2_GATE: now also Q_HS2.4 (G); no longer Q_HS2.1 (G)
- net Q_LS1_GATE: now also Q_LS1.4 (G); no longer Q_LS1.1 (G)
- net Q_LS2_GATE: now also Q_LS2.4 (G); no longer Q_LS2.1 (G)
- new net RSH1_SENSE_HI: RSH1.E1, R_CS1.1, U_ISENSE1.1 (SHUNT_HI)
- new net RSH1_SENSE_LO: C_CS1.2, RSH1.E2, U_DCDC.26 (VOUT1), U_ISENSE1.2 (SHUNT_LO)
- new net RSH2_SENSE_HI: RSH2.E1, R_CS2.1, U_ISENSE2.1 (SHUNT_HI)
- new net RSH2_SENSE_LO: C_CS2.2, RSH2.E2, U_DCDC.5 (VOUT2), U_ISENSE2.2 (SHUNT_LO)
Other:
- note added: "Native KiCad ERC is performed by official KiCad 10.x CI/owner review. Bench Bode/OCP/load-step/thermal Gates remain open."
- note removed: "Native KiCad ERC is performed by CI/owner KiCad 10.0.5. Bench Bode/OCP/load-step/thermal Gates remain open."
- moved on the sheet: L1, L2
